Commit message: intial commit MED18 industrial challenge
The repository contains the initial commit of the MED18 industrial challenge

File: rotors_description/urdf/component_snippets.xacro (robot description, xacro)
@@ -246,19 +246,5 @@
     </gazebo>
   </xacro:macro>
-  <!-- =============================================================== -->
-  <!-- ==================== ROS INTERFACE MACRO ====================== -->
-  <!-- =============================================================== -->
-  <!-- <xacro:macro
-  		name="ros_interface_plugin_macro"
-  		params="namespace">
-    <gazebo>
-      <plugin name="ros_interface_plugin" filename="librotors_gazebo_ros_interface_plugin.so">
-        <robotNamespace>${namespace}</robotNamespace>
-      </plugin>
-    </gazebo>
-  </xacro:macro>-->
-  <!-- =============================================================== -->
-  <!-- ================== MAVLINK INTERFACE MACRO ==================== -->
-  <!-- =============================================================== -->
+  <!-- Macro to add the mavlink interface. -->
   <xacro:macro name="mavlink_interface_macro"
     params="namespace mavlink_sub_topic imu_sub_topic mavlink_pub_topic
@@ -291,5 +277,5 @@
   <xacro:macro name="imu_plugin_macro"
     params="namespace imu_suffix parent_link imu_topic
-      mass_imu_sensor gyroscope_noise_density gyroscope_random_walk
+      mass_imu_sensor gyroscope_noise_density gyroscopoe_random_walk
       gyroscope_bias_correlation_time gyroscope_turn_on_bias_sigma
       accelerometer_noise_density accelerometer_random_walk
@@ -319,5 +305,5 @@
         <imuTopic>${imu_topic}</imuTopic> <!-- (string): name of the sensor output topic and prefix of service names (defaults to imu) -->
         <gyroscopeNoiseDensity>${gyroscope_noise_density}</gyroscopeNoiseDensity> <!-- Gyroscope noise density (two-sided spectrum) [rad/s/sqrt(Hz)] -->
-        <gyroscopeRandomWalk>${gyroscope_random_walk}</gyroscopeRandomWalk> <!-- Gyroscope bias random walk [rad/s/s/sqrt(Hz)] -->
+        <gyroscopeRandomWalk>${gyroscopoe_random_walk}</gyroscopeRandomWalk> <!-- Gyroscope bias random walk [rad/s/s/sqrt(Hz)] -->
         <gyroscopeBiasCorrelationTime>${gyroscope_bias_correlation_time}</gyroscopeBiasCorrelationTime> <!-- Gyroscope bias correlation time constant [s] -->
         <gyroscopeTurnOnBiasSigma>${gyroscope_turn_on_bias_sigma}</gyroscopeTurnOnBiasSigma> <!-- Gyroscope turn on bias standard deviation [rad/s] -->
@@ -497,40 +483,9 @@
     </gazebo>
   </xacro:macro>
-  <!-- Macro to add an air pressure sensor. -->
-  <xacro:macro name="pressure_sensor_plugin_macro"
-    params="namespace pressure_sensor_suffix parent_link pressure_topic
-      mass_pressure_sensor reference_altitude pressure_variance *inertia
-      *origin">
-    <!-- Pressure sensor link -->
-    <link name="${namespace}/pressure_sensor${pressure_sensor_suffix}_link">
-      <inertial>
-        <xacro:insert_block name="inertia" />
-        <mass value="${mass_pressure_sensor}" />  <!-- [kg] -->
-        <origin xyz="0 0 0" rpy="0 0 0" />
-      </inertial>
-    </link>
-    <!-- Pressure sensor joint -->
-    <joint name="${namespace}/pressure_sensor${pressure_sensor_suffix}_joint" type="revolute">
-      <xacro:insert_block name="origin" />
-      <parent link="${parent_link}" />
-      <child link="${namespace}/pressure_sensor${pressure_sensor_suffix}_link" />
-      <limit upper="0" lower="0" effort="0" velocity="0" />
-    </joint>
-    <gazebo>
-      <plugin filename="librotors_gazebo_pressure_plugin.so" name="rotors_gazebo_pressure_sensor${pressure_sensor_suffix}_plugin">
-        <robotNamespace>${namespace}</robotNamespace> <!-- (string, required): ros namespace in which the messages are published -->
-        <linkName>${namespace}/pressure_sensor${pressure_sensor_suffix}_link</linkName> <!-- (string, required): name of the body which holds the pressure sensor -->
-        <pressureTopic>${pressure_topic}</pressureTopic> <!-- (string): name of the sensor output topic and prefix of service names (defaults to 'air_pressure') -->
-        <referenceAltitude>${reference_altitude}</referenceAltitude> <!-- the initial altitude [m] -->
-        <pressureVariance>${pressure_variance}</pressureVariance> <!-- the air pressure variance [Pa^2] -->
-      </plugin>
-    </gazebo>
-  </xacro:macro>
   <!-- Macro to add the wind plugin. -->
   <xacro:macro name="wind_plugin_macro"
     params="namespace xyz_offset wind_direction wind_force_mean
       wind_gust_direction wind_gust_duration wind_gust_start
-      wind_gust_force_mean wind_speed_mean use_custom_static_wind_field
-      custom_wind_field_path">
+      wind_gust_force_mean">
     <gazebo>
       <plugin filename="librotors_gazebo_wind_plugin.so" name="wind_plugin">
@@ -545,7 +500,4 @@
         <windGustStart>${wind_gust_start}</windGustStart> <!-- [s] -->
         <windGustForceMean>${wind_gust_force_mean}</windGustForceMean> <!-- [N] -->
-        <windSpeedMean>${wind_speed_mean}</windSpeedMean> <!-- [m/s] -->
-        <useCustomStaticWindField>${use_custom_static_wind_field}</useCustomStaticWindField>
-        <customWindFieldPath>${custom_wind_field_path}</customWindFieldPath> <!-- from ~/.ros -->
       </plugin>
     </gazebo>
@@ -750,5 +702,5 @@
       mass_imu_sensor="0.015"
       gyroscope_noise_density="0.0003394"
-      gyroscope_random_walk="0.000038785"
+      gyroscopoe_random_walk="0.000038785"
       gyroscope_bias_correlation_time="1000.0"
       gyroscope_turn_on_bias_sigma="0.0087"
@@ -770,5 +722,5 @@
       mass_imu_sensor="0.00001"
       gyroscope_noise_density="0.0"
-      gyroscope_random_walk="0.0"
+      gyroscopoe_random_walk="0.0"
       gyroscope_bias_correlation_time="1000.0"
       gyroscope_turn_on_bias_sigma="0.0"
@@ -820,5 +772,5 @@
       mass_imu_sensor="0.015"
       gyroscope_noise_density="0.0003394"
-      gyroscope_random_walk="0.000038785"
+      gyroscopoe_random_walk="0.000038785"
       gyroscope_bias_correlation_time="1000.0"
       gyroscope_turn_on_bias_sigma="0.0087"
@@ -865,17 +817,4 @@
     </xacro:magnetometer_plugin_macro>
   </xacro:macro>
-  <xacro:macro name="default_pressure_sensor" params="namespace parent_link">
-    <xacro:pressure_sensor_plugin_macro
-      namespace="${namespace}"
-      pressure_sensor_suffix=""
-      parent_link="${parent_link}"
-      pressure_topic="air_pressure"
-      mass_pressure_sensor="0.015"
-      reference_altitude="500.0"
-      pressure_variance="0.0">
-      <inertia ixx="0.00001" ixy="0.0" ixz="0.0" iyy="0.00001" iyz="0.0" izz="0.00001" />
-      <origin xyz="0 0 0" rpy="0 0 0" />
-    </xacro:pressure_sensor_plugin_macro>
-  </xacro:macro>
   <xacro:macro name="default_mavlink_interface" params="namespace imu_sub_topic rotor_count">
     <xacro:mavlink_interface_macro

File: rotors_description/urdf/firefly_base.xacro (robot description, xacro)
@@ -22,6 +22,4 @@
   <!-- Instantiate a controller. -->
   <xacro:controller_plugin_macro namespace="${namespace}" imu_sub_topic="imu" />
-  <!-- Instantiate a ROS message interface -->
-  <!-- <xacro:ros_interface_plugin_macro namespace="${namespace}" />-->
   <xacro:if value="$(arg enable_mavlink_interface)">
     <!-- Instantiate mavlink telemetry interface. -->

File: rotors_description/urdf/fixed_wing_base.xacro (robot description, xacro)
@@ -28,6 +28,5 @@
   <xacro:macro name="fixed_wing_base_macro"
     params="robot_namespace mass length width height color use_mesh_file
-      mesh_file aero_params_yaml vehicle_params_yaml is_input_joystick
-      *origin *inertia">
+      mesh_file *origin *inertia">
     <link name="${robot_namespace}/base_link"></link>
     <joint name="${robot_namespace}/base_joint" type="fixed">
@@ -63,14 +62,4 @@
       <material>Gazebo/${color}</material>
     </gazebo>
-    <!-- Attach fw_dynamics to the base_link -->
-    <gazebo>
-      <plugin filename="librotors_gazebo_fw_dynamics_plugin.so" name="fw_dynamics_plugin">
-        <robotNamespace>${robot_namespace}</robotNamespace>
-        <linkName>${robot_namespace}/base_link</linkName>
-        <aeroParamsYAML>${aero_params_yaml}</aeroParamsYAML>
-        <vehicleParamsYAML>${vehicle_params_yaml}</vehicleParamsYAML>
-        <isInputJoystick>${is_input_joystick}</isInputJoystick>
-      </plugin>
-    </gazebo>
   </xacro:macro>
   <!-- Control surface joint and link -->
@@ -84,5 +73,5 @@
       <parent link="${parent}" />
       <child link="${robot_namespace}/${surface_name}" />
-      <limit upper="0" lower="0" effort="0" velocity="0" />
+      <limit upper="${max_angle}" lower="${min_angle}" effort="0" velocity="0" />
     </joint>
     <link name="${robot_namespace}/${surface_name}">

File: rotors_description/urdf/neo11.xacro (robot description, xacro)
@@ -18,5 +18,5 @@
 <robot name="neo11" xmlns:xacro="http://ros.org/wiki/xacro">
   <!-- Properties -->
-  <xacro:property name="namespace" value="$(arg namespace)" />
+  <xacro:property name="namespace" value="$(arg mav_name)" />
   <xacro:property name="rotor_velocity_slowdown_sim" value="10" />
   <xacro:property name="use_mesh_file" value="true" />

File: rotors_description/urdf/techpod.xacro (robot description, xacro)
@@ -31,5 +31,4 @@
   <xacro:property name="body_height" value="0.303" /> <!-- [m] -->
   <xacro:property name="body_color" value="Gray" />
-  <xacro:property name="body_mesh_file" value="package://rotors_description/meshes/techpod/techpod_body.dae" />
   <!-- Aileron properties -->
   <xacro:property name="aileron_length" value="0.053" /> <!-- [m] -->
@@ -39,6 +38,4 @@
   <xacro:property name="aileron_max_angle" value="0.349066" /> <!-- [rad] -->
   <xacro:property name="aileron_color" value="Red" />
-  <xacro:property name="aileron_left_mesh_file" value="package://rotors_description/meshes/techpod/techpod_aileron_left.dae" />
-  <xacro:property name="aileron_right_mesh_file" value="package://rotors_description/meshes/techpod/techpod_aileron_right.dae" />
   <!-- Elevator properties -->
   <xacro:property name="elevator_length" value="0.051" /> <!-- [m] -->
@@ -48,5 +45,4 @@
   <xacro:property name="elevator_max_angle" value="0.349066" /> <!-- [rad] -->
   <xacro:property name="elevator_color" value="Blue" />
-  <xacro:property name="elevator_mesh_file" value="package://rotors_description/meshes/techpod/techpod_elevator.dae" />
   <!-- Flap properties -->
   <xacro:property name="flap_length" value="0.076" /> <!-- [m] -->
@@ -56,6 +52,4 @@
   <xacro:property name="flap_max_angle" value="0.0" /> <!-- [rad] -->
   <xacro:property name="flap_color" value="Yellow" />
-  <xacro:property name="flap_left_mesh_file" value="package://rotors_description/meshes/techpod/techpod_flap_left.dae" />
-  <xacro:property name="flap_right_mesh_file" value="package://rotors_description/meshes/techpod/techpod_flap_right.dae" />
   <!-- Rudder properties -->
   <xacro:property name="rudder_length" value="0.129" />
@@ -65,5 +59,4 @@
   <xacro:property name="rudder_max_angle" value="0.349066" />
   <xacro:property name="rudder_color" value="Orange" />
-  <xacro:property name="rudder_mesh_file" value="package://rotors_description/meshes/techpod/techpod_rudder.dae" />
   <!-- Propeller properties -->
   <xacro:property name="propeller_direction" value="cw" />
@@ -71,5 +64,4 @@
   <xacro:property name="propeller_height" value="0.003" />
   <xacro:property name="propeller_color" value="Gray" />
-  <xacro:property name="propeller_mesh_file" value="package://rotors_description/meshes/propeller_${propeller_direction}.dae" />
   <!-- Inertia of the main body -->
   <xacro:property name="body_inertia">
@@ -107,8 +99,5 @@
     color="${body_color}"
     use_mesh_file="${use_mesh}"
-    mesh_file="${body_mesh_file}"
-    aero_params_yaml="$(arg aero_params_yaml_file)"
-    vehicle_params_yaml="$(arg vehicle_params_yaml_file)"
-    is_input_joystick="$(arg is_input_joystick)">
+    mesh_file="package://rotors_description/meshes/techpod/techpod_body.dae">
     <origin xyz="0 0 0" rpy="0 0 0" />
     <xacro:insert_block name="body_inertia" />
@@ -124,5 +113,5 @@
     color="${aileron_color}"
     use_mesh_file="${use_mesh}"
-    mesh_file="${aileron_left_mesh_file}"
+    mesh_file="package://rotors_description/meshes/techpod/techpod_aileron_left.dae"
     surface_length="${aileron_length}"
     surface_width="${aileron_width}"
@@ -142,5 +131,5 @@
     color="${aileron_color}"
     use_mesh_file="${use_mesh}"
-    mesh_file="${aileron_right_mesh_file}"
+    mesh_file="package://rotors_description/meshes/techpod/techpod_aileron_right.dae"
     surface_length="${aileron_length}"
     surface_width="${aileron_width}"
@@ -161,5 +150,5 @@
     color="${elevator_color}"
     use_mesh_file="${use_mesh}"
-    mesh_file="${elevator_mesh_file}"
+    mesh_file="package://rotors_description/meshes/techpod/techpod_elevator.dae"
     surface_length="${elevator_length}"
     surface_width="${elevator_width}"
@@ -180,5 +169,5 @@
     color="${flap_color}"
     use_mesh_file="${use_mesh}"
-    mesh_file="${flap_left_mesh_file}"
+    mesh_file="package://rotors_description/meshes/techpod/techpod_flap_left.dae"
     surface_length="${flap_length}"
     surface_width="${flap_width}"
@@ -198,5 +187,5 @@
     color="${flap_color}"
     use_mesh_file="${use_mesh}"
-    mesh_file="${flap_right_mesh_file}"
+    mesh_file="package://rotors_description/meshes/techpod/techpod_flap_right.dae"
     surface_length="${flap_length}"
     surface_width="${flap_width}"
@@ -217,5 +206,5 @@
     color="${rudder_color}"
     use_mesh_file="${use_mesh}"
-    mesh_file="${rudder_mesh_file}"
+    mesh_file="package://rotors_description/meshes/techpod/techpod_rudder.dae"
     surface_length="${rudder_length}"
     surface_width="${rudder_width}"
@@ -235,5 +224,5 @@
     color="${propeller_color}"
     use_mesh_file="${use_mesh}"
-    mesh_file="${propeller_mesh_file}">
+    mesh_file="package://rotors_description/meshes/propeller_${propeller_direction}.dae">
     <origin xyz="-0.025 0 0.15" rpy="0 ${-0.5*PI} 0" />
     <xacro:insert_block name="propeller_inertia" />

File: rotors_description/urdf/techpod_base.xacro (robot description, xacro)
@@ -22,6 +22,4 @@
   <!-- Mount a magnetometer. -->
   <xacro:default_magnetometer namespace="${namespace}" parent_link="${namespace}/base_link" />
-  <!-- Mount a pressure sensor. -->
-  <xacro:default_pressure_sensor namespace="${namespace}" parent_link="${namespace}/base_link" />
   <xacro:if value="$(arg enable_ground_truth)">
     <xacro:ground_truth_imu_and_odometry namespace="${namespace}" parent_link="${namespace}/base_link_inertia" />

Commit message: Change in the component_snippets file
Some changes in the component_snippets file. Now, the inertial sensors work, i.e., virtual odometry sensor and IMU

File: rotors_description/urdf/component_snippets.xacro (robot description, xacro)
@@ -17,5 +17,4 @@
 -->
 <robot xmlns:xacro="http://ros.org/wiki/xacro">
-  <xacro:property name="pi" value="3.14159265359" />
   <!-- Macro to add logging to a bag file. -->
   <xacro:macro name="bag_plugin_macro"
@@ -277,6 +276,6 @@
   <xacro:macro name="imu_plugin_macro"
     params="namespace imu_suffix parent_link imu_topic
-      mass_imu_sensor gyroscope_noise_density gyroscopoe_random_walk
-      gyroscope_bias_correlation_time gyroscope_turn_on_bias_sigma
+      mass_imu_sensor measurement_divisor measurement_delay gyroscope_noise_density
+      gyroscope_random_walk gyroscope_bias_correlation_time gyroscope_turn_on_bias_sigma
       accelerometer_noise_density accelerometer_random_walk
       accelerometer_bias_correlation_time accelerometer_turn_on_bias_sigma
@@ -305,5 +304,7 @@
         <imuTopic>${imu_topic}</imuTopic> <!-- (string): name of the sensor output topic and prefix of service names (defaults to imu) -->
         <gyroscopeNoiseDensity>${gyroscope_noise_density}</gyroscopeNoiseDensity> <!-- Gyroscope noise density (two-sided spectrum) [rad/s/sqrt(Hz)] -->
-        <gyroscopeRandomWalk>${gyroscopoe_random_walk}</gyroscopeRandomWalk> <!-- Gyroscope bias random walk [rad/s/s/sqrt(Hz)] -->
+        <measurementDivisor>${measurement_divisor}</measurementDivisor> <!-- only every (seq % measurementDivisor) == 0 measurement is published [int] -->
+        <measurementDelay>${measurement_delay}</measurementDelay> <!-- time that measurement gets held back before it's published in [simulation cycles (int)] -->
+        <gyroscopeRandomWalk>${gyroscope_random_walk}</gyroscopeRandomWalk> <!-- Gyroscope bias random walk [rad/s/s/sqrt(Hz)] -->
         <gyroscopeBiasCorrelationTime>${gyroscope_bias_correlation_time}</gyroscopeBiasCorrelationTime> <!-- Gyroscope bias correlation time constant [s] -->
         <gyroscopeTurnOnBiasSigma>${gyroscope_turn_on_bias_sigma}</gyroscopeTurnOnBiasSigma> <!-- Gyroscope turn on bias standard deviation [rad/s] -->
@@ -676,6 +677,6 @@
         child_frame_id="${namespace}/base_link"
         mass_odometry_sensor="0.00001"
+        measurement_delay="0"
         measurement_divisor="1"
-        measurement_delay="0"
         unknown_delay="0.0"
         noise_normal_position="0 0 0"
@@ -702,7 +703,9 @@
       mass_imu_sensor="0.015"
       gyroscope_noise_density="0.0003394"
-      gyroscopoe_random_walk="0.000038785"
+      gyroscope_random_walk="0.000038785"
       gyroscope_bias_correlation_time="1000.0"
       gyroscope_turn_on_bias_sigma="0.0087"
+      measurement_delay="0"
+      measurement_divisor="1"
       accelerometer_noise_density="0.004"
       accelerometer_random_walk="0.006"
@@ -721,6 +724,8 @@
       imu_topic="ground_truth/imu"
       mass_imu_sensor="0.00001"
+      measurement_delay="0"
+      measurement_divisor="1"
       gyroscope_noise_density="0.0"
-      gyroscopoe_random_walk="0.0"
+      gyroscope_random_walk="0.0"
       gyroscope_bias_correlation_time="1000.0"
       gyroscope_turn_on_bias_sigma="0.0"
@@ -745,6 +750,6 @@
       child_frame_id="${namespace}/base_link"
       mass_odometry_sensor="0.00001"
+      measurement_delay="0"
       measurement_divisor="1"
-      measurement_delay="0"
       unknown_delay="0.0"
       noise_normal_position="0 0 0"
@@ -771,6 +776,8 @@
       imu_topic="imu"
       mass_imu_sensor="0.015"
+      measurement_delay="0"
+      measurement_divisor="1"
       gyroscope_noise_density="0.0003394"
-      gyroscopoe_random_walk="0.000038785"
+      gyroscope_random_walk="0.000038785"
       gyroscope_bias_correlation_time="1000.0"
       gyroscope_turn_on_bias_sigma="0.0087"
